File: hardware/rs485-extension.kicad_pcb (KiCad board)
At the start: 2 copper layers, 40 x 40 mm, 27 parts, among them J1 STACK-UP-HIGH, J2 STACK-DOWN, J3 STACK-UP-HIGH, J4 STACK-DOWN, K1 grey, SW1 TER, U1 M24C64, U2 ADM3485, U3 DRILL, U4 DRILL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

Commit message: drc check executed
Parts:
- C1, C2, D1, R1, R3: footprint kicad-libraries:0603 -> kicad-libraries:0603E
- moved R1 0.12 mm to (147.1, 81.0)

Commit message: Add 3d information (tbc)
Parts:
- C1, C2: footprint kicad-libraries:0603E -> kicad-libraries:C0603
- D1: footprint kicad-libraries:0603E -> kicad-libraries:D0603
- Fiducial_Mark (x4): footprint Fiducial_Mark -> kicad-libraries:Fiducial_Mark
- R1, R3: footprint kicad-libraries:0603E -> kicad-libraries:R0603
- R2: footprint kicad-libraries:D0603 -> kicad-libraries:R0603
- VAL: footprint WEEE_7mm -> kicad-libraries:WEEE_7mm
- VAL: footprint CE_5mm -> kicad-libraries:CE_5mm
Connections:
- FILTER1 pad 10: (no net) -> Net-(FILTER1-Pad10)
- FILTER1 pad 12: (no net) -> Net-(FILTER1-Pad12)
- FILTER1 pad 14: (no net) -> Net-(FILTER1-Pad14)
- FILTER1 pad 3: (no net) -> Net-(FILTER1-Pad3)
- FILTER1 pad 5: (no net) -> Net-(FILTER1-Pad5)
- FILTER1 pad 7: (no net) -> Net-(FILTER1-Pad7)
- J1 pad 25: (no net) -> Net-(J1-Pad25)
- J1 pad 27: (no net) -> Net-(J1-Pad27)
- J1 pad 29: (no net) -> Net-(J1-Pad29)
- J2 pad 21: (no net) -> Net-(J2-Pad21)
- J2 pad 23: (no net) -> Net-(J2-Pad23)
- L1 pad 4: (no net) -> Net-(L1-Pad4)
- L1 pad 5: (no net) -> Net-(L1-Pad5)
- SW1 pad 3: (no net) -> Net-(SW1-Pad3)
- SW1 pad 4: (no net) -> Net-(SW1-Pad4)
- SW1 pad 5: (no net) -> Net-(SW1-Pad5)
- SW1 pad 6: (no net) -> Net-(SW1-Pad6)
- U1 pad 7: (no net) -> Net-(U1-Pad7)
